File: hardware/picostepknobs.brd (EAGLE design)
At the start: 177.8 x 81.3 mm, 48 parts, among them IC1 4051D, J1 AUDIO-JACK-TRRS, J2 AUDIO-JACK-TRRS, P1 10k, P2 10k, P3 10k, P4 10k, P5 10k, P6 10k, P7 10k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

Commit message: brd layout
Parts:
- added C10, C11, C12, C9: 100n, rcl:C0805
- added LED10, LED11, LED12, LED9: WS2812B3535, todstuff2023:LED3535
- renumbered MODULE1 to PCM5102A
Connections:
- new net N$14: LED10.1, LED9.3
- new net N$15: LED10.3, LED11.1
- new net N$16: LED11.3, LED12.1
- new net N$17: LED8.3, LED9.1
- net +3V3: now also C10.1, C11.1, C12.1, C9.1, LED10.2, LED11.2, LED12.2, LED9.2
- net GND: now also C10.2, C11.2, C12.2, C9.2, LED10.4, LED11.4, LED12.4, LED9.4
Routing:
- net N$17: track 0.00 -> 117.2 mm, vias 0 -> 2
- net GND: track 136.2 -> 165.6 mm, vias 1 -> 3
- net N$15: track 0.00 -> 8.95 mm
- net N$14: track 0.00 -> 4.88 mm
- net N$16: track 0.00 -> 4.88 mm
- net SW9: track 100.3 -> 102.9 mm
- net POT_IN: track 97.0 -> 95.2 mm
- net N$48: track 14.3 -> 13.3 mm
- net DISP_RES: track 71.2 -> 70.3 mm
- net SW11: track 55.2 -> 56.0 mm
