File: hardware/picostepknobs.sch (EAGLE design)
At the start: 48 parts, among them IC1 4051D, J1 AUDIO-JACK-TRRS, J2 AUDIO-JACK-TRRS, P1 10k, P2 10k, P3 10k, P4 10k, P5 10k, P6 10k, P7 10k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

Commit message: brd layout
Parts:
- removed MODULE1: I2S_PCM_51XX_SOUNDCARD, PCM5102A:I2S_PCM_51XX_SOUNDCARD
- added C10, C11, C12, C9: 100n, rcl:C-EUC0805
- added LED10, LED11, LED12, LED9: WS2812B3535, todstuff2023:WS2812B3535
- added PCM5102A: I2S_PCM_51XX_SOUNDCARD, PCM5102A:I2S_PCM_51XX_SOUNDCARD
Connections:
- new net N$14: LED10.DI, LED9.DO
- new net N$15: LED10.DO, LED11.DI
- new net N$16: LED11.DO, LED12.DI
- new net N$17: LED8.DO, LED9.DI
- net +3V3: now also C10.1, C11.1, C12.1, C9.1, LED10.VDD, LED11.VDD, LED12.VDD, LED9.VDD, PCM5102A.VIN; no longer MODULE1.VIN
- net GND: now also C10.2, C11.2, C12.2, C9.2, LED10.GND, LED11.GND, LED12.GND, LED9.GND, PCM5102A.GND, PCM5102A.SCK; no longer MODULE1.GND, MODULE1.SCK
- net I2S_BCLK: now also PCM5102A.BCK; no longer MODULE1.BCK
- net I2S_DIN: now also PCM5102A.DIN; no longer MODULE1.DIN
- net I2S_LCK: now also PCM5102A.LCK; no longer MODULE1.LCK
Other:
- note added: "MIDI TRS-A IN"
- note added: "PCM5012A"
- note added: "https://github.com/todbot/picostepknobs"
- note removed: "https://github.com/todbot/picostepseq"
- moved on the sheet: DISP1
